Commit message: Add SLAM Toolbox integration and web UI for robot control
Replaces GMapping with SLAM Toolbox for improved mapping and localization,
including new configuration and launch files tailored to the Husky UR5
platform and Gazebo simulation.

Introduces a Flask-based web interface with command queueing for safe
multi-threaded ROS operation. Enables semantic map saving, pose management,
and remote control through a browser.

Updates navigation parameters for better indoor performance, costmap tuning,
and robot footprint accuracy. Adds scripts for initial pose publication and
semantic map shifting to streamline workflows.

Removes deprecated or unused files to clean up the codebase and adds a
sample Gazebo model for simulation.

Improves robustness and flexibility for both simulation and real-robot
scenarios.

File: src/husky_ur5_moveit_config/config/gazebo_husky_ur5.urdf (robot description, URDF)
Before this commit: robot husky_ur5, 33 links, 32 joints
Links:
- link base_laser_mount: mass 0.1 -> None; geometry 
Joints:
- joint base_laser_joint: origin xyz=0.0352 0 0.0566 rpy=3.14159 0 0 -> xyz=0.055 0 0.0365 rpy=0 0 0
- joint base_laser_mount_joint: origin xyz=0.3 0.0 0.0 rpy=0.0 0.0 0.0 -> xyz=0.3 0.0 -0.10 rpy=0.0 0.0 0.0

File: src/mobile_manipulator/urdf/husky_ur5.urdf.xacro (robot description, xacro)
@@ -3,10 +3,12 @@
   <xacro:include filename="$(find husky_description)/urdf/husky.urdf.xacro" />
   <xacro:include filename="$(find husky_description)/urdf/accessories/sick_lms1xx_mount.urdf.xacro" />
+  <!-- LiDAR lowered from 37.7 cm to 25.7 cm above ground to detect low obstacles.
+       tower="0" removes the raised bracket; z=-0.10 drops it 10 cm below top_plate. -->
   <xacro:sick_lms1xx_mount prefix="base"
     parent="top_plate_link"
     topic="/front/scan"
     robot_namespace="/"
-    tower="1">
-    <origin xyz="0.3 0.0 0.0" rpy="0.0 0.0 0.0" />
+    tower="0">
+    <origin xyz="0.3 0.0 -0.10" rpy="0.0 0.0 0.0" />
   </xacro:sick_lms1xx_mount>
   <xacro:include filename="$(find ur_description)/urdf/inc/ur_macro.xacro"/>
@@ -53,5 +55,5 @@
     <parent link="ur5_tool0" />
     <child link="realsense_camera_link" />
-    <origin xyz="0.0 0.05 0.0" rpy="0.0 -1.57 1.57" />
+    <origin xyz="0.0 0.05 0.0" rpy="0.0 -1.57 -1.57" />
   </joint>
   <!-- Dummy Link & Joint -->

Commit message: Refactor MasterControl for improved object detection and manipulation
- Enhanced the scan_with_arm method to include bounding box width in detection results.
- Updated get_3d_coordinates to utilize bounding box width for more accurate depth calculations.
- Improved execute_pick to refine grasp poses based on re-detection of objects.
- Added scene collision updates to dynamically adjust for detected objects.
- Modified URDF to correct the joint origin for the robot's camera frame.
- Introduced a marker publisher for visual debugging in RViz.
- Adjusted arm joint configurations for better scanning positions.

File: src/husky_ur5_moveit_config/config/gazebo_husky_ur5.urdf (robot description, URDF)
Before this commit: robot husky_ur5, 33 links, 32 joints
Joints:
- joint camera_to_wrist: origin xyz=0.0 0.05 0.0 rpy=0.0 -1.57 1.57 -> xyz=0.0 0.05 0.0 rpy=0.0 -1.57 -1.57
- joint husky_to_ur5_joint: origin xyz=-0.1 0.0 0.0 rpy=0.0 0.0 0.0 -> xyz=0.1 0.0 0.0 rpy=0.0 0.0 0.0

File: src/mobile_manipulator/urdf/husky_ur5.urdf.xacro (robot description, xacro)
@@ -23,5 +23,5 @@
     <parent link="top_plate_link" />
     <child link="ur5_base_link" />
-    <origin xyz="-0.1 0.0 0.0" rpy="0.0 0.0 0.0" />
+    <origin xyz="0.1 0.0 0.0" rpy="0.0 0.0 0.0" />
   </joint>
   <!-- Gripper -->
@@ -57,9 +57,18 @@
     <origin xyz="0.0 0.05 0.0" rpy="0.0 -1.57 -1.57" />
   </joint>
-  <!-- Dummy Link & Joint -->
+  <!--
+    Optical-frame "dummy" link (no mass / visual / collision — intentional).
+    REP-103 convention: Z forward (into scene), X right, Y down.
+    rpy="-π/2 0 -π/2" rotates the camera body frame (Z forward, Y up) to the
+    optical frame (Z forward, Y down). This must match the convention assumed by
+    the pinhole back-projection in get_3d_coordinates and by libgazebo_ros_openni_kinect
+    (frameName = realsense_camera_optical_frame).  Do NOT change this transform
+    without updating the back-projection formula.
+  -->
   <link name="realsense_camera_optical_frame" />
   <joint name="camera_optical_joint" type="fixed">
-    <origin xyz="0 0 0" rpy="-1.5708 0 -1.5708" /> <parent link="realsense_camera_link" />
+    <parent link="realsense_camera_link" />
     <child link="realsense_camera_optical_frame" />
+    <origin xyz="0 0 0" rpy="-1.5708 0 -1.5708" />
   </joint>
   <gazebo reference="realsense_camera_link">

Commit message: Remove beginner_tutorials package files and add grasp fix plugin to gazebo_husky_ur5.urdf for improved object handling

File: src/husky_ur5_moveit_config/config/gazebo_husky_ur5.urdf (robot description, URDF)
Before this commit: robot husky_ur5, 33 links, 32 joints
Links:
- added link base_ballast, mass 30.0
- link base_link: mass 0.1 -> None
- link top_plate_link: mass 0.1 -> None
Joints:
- added joint base_ballast_joint: type fixed, parent base_link, child base_ballast, origin xyz=0 0 0 rpy=0 0 0

File: src/mobile_manipulator/urdf/husky_ur5.urdf.xacro (robot description, xacro)
@@ -25,4 +25,23 @@
     <origin xyz="0.1 0.0 0.0" rpy="0.0 0.0 0.0" />
   </joint>
+  <!-- Virtual ballast: simulates the Husky's rear battery bank.
+       The stock inertial_link iyy (1.74 kg⋅m²) is less than half the
+       theoretical value for the chassis dimensions, leaving the base on the
+       edge of tipping when the arm is extended.  30 kg placed 0.15 m behind
+       and 0.08 m below base_link shifts the CoM rearward and raises iyy
+       enough to keep the robot stable through the full grasp motion. -->
+  <link name="base_ballast">
+    <inertial>
+      <mass value="30.0" />
+      <origin xyz="-0.15 0.0 -0.08" rpy="0 0 0" />
+      <inertia ixx="1.5" ixy="0" ixz="0"
+               iyy="3.0" iyz="0" izz="3.0" />
+    </inertial>
+  </link>
+  <joint name="base_ballast_joint" type="fixed">
+    <parent link="base_link" />
+    <child link="base_ballast" />
+    <origin xyz="0 0 0" rpy="0 0 0" />
+  </joint>
   <!-- Gripper -->
   <xacro:include filename="$(find robotiq_description)/urdf/robotiq_hande_gripper.urdf.xacro" />
@@ -31,5 +50,24 @@
     <origin xyz="0 0 0" rpy="0 0 0"/>
   </xacro:robotiq_hande_gripper>
-<link name="realsense_camera_link">
+  <!-- Grasp fix: creates a virtual joint between gripper and object when both
+       fingers make opposing contact, preventing the object from flying away. -->
+  <gazebo>
+    <plugin filename="libgazebo_grasp_fix.so" name="gazebo_grasp_fix">
+      <arm>
+        <arm_name>hande_gripper</arm_name>
+        <palm_link>ur5_wrist_3_link</palm_link>
+        <gripper_link>hande_left_finger</gripper_link>
+        <gripper_link>hande_right_finger</gripper_link>
+      </arm>
+      <forces_angle_tolerance>100</forces_angle_tolerance>
+      <update_rate>90</update_rate>
+      <grip_count_threshold>1</grip_count_threshold>
+      <max_grip_count>8</max_grip_count>
+      <release_tolerance>0.005</release_tolerance>
+      <disable_collisions_on_attach>false</disable_collisions_on_attach>
+      <contact_topic>__default_topic__</contact_topic>
+    </plugin>
+  </gazebo>
+  <link name="realsense_camera_link">
     <visual>
       <geometry>
