Commit message: Outdoor air-ground system + collaboration repo setup
Features:
- Dual-EKF outdoor localization: navsat_transform + global EKF (map->odom)
  fusing the Husky's simulated GPS, plus transform_timeout tuning
- Gripper upgrade Hand-E (50 mm) -> Robotiq 2F-140 (140 mm): URDF, grasp-fix
  plugin, SRDF collision matrix, MoveIt + controller configs, and the
  master_control pick/place logic (revolute finger_joint, diameter->angle map)
- outdoor_city.world: 500 m heightmap terrain + 130-tree mountain forest
- generate_forest.py: reproducible, slope-aware tree placement (seats trees on
  the canopy-footprint max so slopes never bury them)
- spawn_outdoor_city.launch wiring world + robot + GPS/EKF + controllers

Repo setup for collaboration:
- Vendor robotiq (was a broken gitlink -> empty on clone)
- aws-robomaker (indoor-only, ~131 MB) kept local but gitignored, not shared
- Keep only the 13 Gazebo models our worlds use; drop ~380 unused (~1.3 GB)
- gitignore hardware-specific TensorRT *.engine; stop tracking a stale *.pyc
- Add .gitattributes (LF normalization + binary handling for meshes/images)

Co-Authored-By: Claude Opus 4.8 <noreply@anthropic.com>

File: src/husky_ur5_moveit_config/config/gazebo_husky_ur5.urdf (robot description, URDF)
Before this commit: robot husky_ur5, 34 links, 33 joints
Links:
- removed link hand_e_link
- removed link hande_left_finger
- removed link hande_right_finger
- added link left_inner_finger, mass 0.0104003125914103; collision mesh filename=package://robotiq_description/meshes/collision/robotiq_arg2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; visual mesh filename=package://robotiq_description/meshes/visual/robotiq_arg2f_1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
- added link left_inner_finger_pad; collision box size=0.025 0.06 0.0075; visual box size=0.027 0.065 0.0075
- added link left_inner_knuckle, mass 0.0271177346495152; collision mesh filename=package://robotiq_description/meshes/collision/robotiq_arg2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; visual mesh filename=package://robotiq_description/meshes/visual/robotiq_arg2f_1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
- added link left_outer_finger, mass 0.022614240507152; collision mesh filename=package://robotiq_description/meshes/collision/robotiq_arg2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; visual mesh filename=package://robotiq_description/meshes/visual/robotiq_arg2f_1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
- added link left_outer_knuckle, mass 0.00853198276973456; collision mesh filename=package://robotiq_description/meshes/collision/robotiq_arg2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; visual mesh filename=package://robotiq_description/meshes/visual/robotiq_arg2f_1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
- added link right_inner_finger, mass 0.0104003125914103; collision mesh filename=package://robotiq_description/meshes/collision/robotiq_arg2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; visual mesh filename=package://robotiq_description/meshes/visual/robotiq_arg2f_1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
- added link right_inner_finger_pad; collision box size=0.025 0.06 0.0075; visual box size=0.027 0.065 0.0075
- added link right_inner_knuckle, mass 0.0271177346495152; collision mesh filename=package://robotiq_description/meshes/collision/robotiq_arg2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; visual mesh filename=package://robotiq_description/meshes/visual/robotiq_arg2f_1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
- added link right_outer_finger, mass 0.022614240507152; collision mesh filename=package://robotiq_description/meshes/collision/robotiq_arg2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; visual mesh filename=package://robotiq_description/meshes/visual/robotiq_arg2f_1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
- added link right_outer_knuckle, mass 0.00853198276973456; collision mesh filename=package://robotiq_description/meshes/collision/robotiq_arg2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; visual mesh filename=package://robotiq_description/meshes/visual/robotiq_arg2f_1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
- added link robotiq_140_base_link
- added link robotiq_arg2f_base_link, mass 0.22652; collision mesh filename=package://robotiq_description/meshes/collision/robotiq_arg2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; visual mesh filename=package://robotiq_description/meshes/visual/robotiq_arg2f_b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
Joints:
- removed joint hande_left_finger_joint
- removed joint hande_right_finger_joint
- removed joint robotiq_hande_base_joint
- added joint finger_joint: type revolute, parent robotiq_arg2f_base_link, child left_outer_knuckle, origin xyz=0 -0.030601 0.054905 rpy=2.2957963267948966 0 0, axis -1 0 0, limit lower=0 upper=0.725 effort=1000 velocity=2.0
- added joint left_inner_finger_joint: type revolute, parent left_outer_finger, child left_inner_finger, origin xyz=0 0.0817554015893473 -0.0282203446692936 rpy=-0.725 0 0, axis 1 0 0, limit lower=-0.8757 upper=0.8757 effort=1000 velocity=2.0, mimic joint=finger_joint multiplier=1 offset=0
- added joint left_inner_finger_pad_joint: type fixed, parent left_inner_finger, child left_inner_finger_pad, origin xyz=0 0.0457554015893473 -0.0272203446692936 rpy=0 0 0, axis 0 0 1
- added joint left_inner_knuckle_joint: type revolute, parent robotiq_arg2f_base_link, child left_inner_knuckle, origin xyz=0 -0.0127 0.06142 rpy=2.2957963267948966 0 0.0, axis 1 0 0, limit lower=-0.8757 upper=0.8757 effort=1000 velocity=2.0, mimic joint=finger_joint multiplier=-1 offset=0
- added joint left_outer_finger_joint: type fixed, parent left_outer_knuckle, child left_outer_finger, origin xyz=0 0.01821998610742 0.0260018192872234 rpy=0 0 0, axis 1 0 0
- added joint right_inner_finger_joint: type revolute, parent right_outer_finger, child right_inner_finger, origin xyz=0 0.0817554015893473 -0.0282203446692936 rpy=-0.725 0 0, axis 1 0 0, limit lower=-0.8757 upper=0.8757 effort=1000 velocity=2.0, mimic joint=finger_joint multiplier=1 offset=0
- added joint right_inner_finger_pad_joint: type fixed, parent right_inner_finger, child right_inner_finger_pad, origin xyz=0 0.0457554015893473 -0.0272203446692936 rpy=0 0 0, axis 0 0 1
- added joint right_inner_knuckle_joint: type revolute, parent robotiq_arg2f_base_link, child right_inner_knuckle, origin xyz=0 0.0127 0.06142 rpy=2.2957963267948966 0 -3.141592653589793, axis 1 0 0, limit lower=-0.8757 upper=0.8757 effort=1000 velocity=2.0, mimic joint=finger_joint multiplier=-1 offset=0
- added joint right_outer_finger_joint: type fixed, parent right_outer_knuckle, child right_outer_finger, origin xyz=0 0.01821998610742 0.0260018192872234 rpy=0 0 0, axis 1 0 0
- added joint right_outer_knuckle_joint: type revolute, parent robotiq_arg2f_base_link, child right_outer_knuckle, origin xyz=0 0.030601 0.054905 rpy=2.2957963267948966 0 3.141592653589793, axis 1 0 0, limit lower=-0.725 upper=0.725 effort=1000 velocity=2.0, mimic joint=finger_joint multiplier=-1 offset=0
- added joint robotiq_140_base_joint: type fixed, parent ur5_tool0, child robotiq_140_base_link, origin xyz=0 0 0 rpy=0 0 0
- added joint robotiq_arg2f_base_joint: type fixed, parent robotiq_140_base_link, child robotiq_arg2f_base_link, origin xyz=0 0 0 rpy=3.141592653589793 -1.5707963267948966 0

File: src/mobile_manipulator/urdf/husky_ur5.urdf.xacro (robot description, xacro)
@@ -45,18 +45,26 @@
   </joint>
   <!-- Gripper -->
-  <xacro:include filename="$(find robotiq_description)/urdf/robotiq_hande_gripper.urdf.xacro" />
-  <!-- Attach the robotiq hand-e gripper -->
-  <xacro:robotiq_hande_gripper prefix="" parent="ur5_tool0" >
+  <!-- Robotiq 2F-140 parallel-jaw gripper: 140 mm max stroke (~3x the Hand-E's
+       50 mm), enabling grasps of larger outdoor objects. Single actuated joint
+       finger_joint (revolute, 0 rad = open, 0.7 rad = closed); all other finger
+       joints mimic it via the gazebo_mimic_joint plugins defined in the macro. -->
+  <xacro:include filename="$(find robotiq_description)/urdf/robotiq_140_gripper.urdf.xacro" />
+  <xacro:robotiq_140_gripper prefix="" parent="ur5_tool0" >
     <origin xyz="0 0 0" rpy="0 0 0"/>
-  </xacro:robotiq_hande_gripper>
+  </xacro:robotiq_140_gripper>
   <!-- Grasp fix: creates a virtual joint between gripper and object when both
        fingers make opposing contact, preventing the object from flying away. -->
   <gazebo>
     <plugin filename="libgazebo_grasp_fix.so" name="gazebo_grasp_fix">
+      <!-- palm_link must be a link that survives Gazebo's fixed-joint lumping.
+           robotiq_arg2f_base_link is attached by a fixed joint and gets merged
+           into the UR5 wrist, so we use ur5_wrist_3_link as the palm (as the
+           Hand-E setup did). The inner_finger links are joined by revolute joints
+           and survive; they also absorb the fixed-jointed finger-pad collisions. -->
       <arm>
-        <arm_name>hande_gripper</arm_name>
+        <arm_name>robotiq_140</arm_name>
         <palm_link>ur5_wrist_3_link</palm_link>
-        <gripper_link>hande_left_finger</gripper_link>
-        <gripper_link>hande_right_finger</gripper_link>
+        <gripper_link>left_inner_finger</gripper_link>
+        <gripper_link>right_inner_finger</gripper_link>
       </arm>
       <forces_angle_tolerance>100</forces_angle_tolerance>
