Commit message: fix(gripper initial pose): update move_it config, fix initial pose issue by pause gazebo @ booting

File: src/mobile_manipulator/urdf/husky_ur5.urdf.xacro (robot description, xacro)
@@ -51,5 +51,5 @@
   <xacro:include filename="$(find robotiq_description)/urdf/robotiq_140_gripper.urdf.xacro" />
   <xacro:robotiq_140_gripper prefix="" parent="ur5_tool0" >
-    <origin xyz="0 0 0" rpy="0 0 0"/>
+    <origin xyz="0 0 0" rpy="0 -1.57 1.57"/>
   </xacro:robotiq_140_gripper>
   <!-- Grasp fix: creates a virtual joint between gripper and object when both

Commit message: feat(egocentric):Implement egocentric UGV navigation and UAV map anchoring
Establishes a full-egocentric navigation framework for the UGV utilizing LiDAR-inertial odometry, removing the need for a global map frame or GPS in the active tracking loop.

To support cooperative air-ground operations, a capture-once anchor node is added to dynamically bind the UAV's local mapping frame to the UGV's drift-free odometry frame. This framework also integrates a self-filtering pipeline to clear the robot's arm from sensor scans, provides an adapter to feed elevation maps directly into the local planner as a unified cost source, and introduces helper utilities and launch files to coordinate the entire egocentric stack.

File: src/mobile_manipulator/urdf/husky_ur5.urdf.xacro (robot description, xacro)
@@ -12,4 +12,83 @@
     <origin xyz="0.3 0.0 -0.10" rpy="0.0 0.0 0.0" />
   </xacro:sick_lms1xx_mount>
+  <!-- ===== Velodyne VLP-16 3D LiDAR (egocentric LIO + terrain perception) =====
+       Mounted on a short mast at the REAR of the top plate (x=-0.30) and raised
+       0.40 m. The UR5 base sits at +0.10 and its ~0.85 m reach covers the whole
+       plate, so no flat-plate spot is outside the arm's envelope; placing the
+       LiDAR behind where the arm actually folds (stow) and reaches (forward
+       grasps) keeps the sensor clear of the arm while still giving an elevated
+       360° sweep. Child scan frame = "velodyne", cloud topic = /velodyne_points.
+       Single exteroceptive sensor for the LIO frontend (DLIO/FAST-LIO) + CMU
+       terrain/local planner.
+       gpu:=true uses the GPU ray plugin (libgazebo_ros_velodyne_gpu_laser): the
+       CPU multiray sensor produces no cloud for a 16-layer Velodyne under
+       gzserver. A GPU + GL context (DISPLAY) is required; this machine has both.
+       The arm may still clip the FoV — robot_body_filter removes it downstream. -->
+  <!-- thin support mast: top_plate -> 0.40 m up at x=-0.30 (behind the arm) -->
+  <link name="velodyne_mast_link">
+    <visual>
+      <origin xyz="0 0 0.20" rpy="0 0 0"/>
+      <geometry><cylinder radius="0.025" length="0.40"/></geometry>
+      <material name="mast_grey"><color rgba="0.2 0.2 0.2 1"/></material>
+    </visual>
+    <collision>
+      <origin xyz="0 0 0.20" rpy="0 0 0"/>
+      <geometry><cylinder radius="0.025" length="0.40"/></geometry>
+    </collision>
+    <inertial>
+      <mass value="0.3"/>
+      <origin xyz="0 0 0.20" rpy="0 0 0"/>
+      <inertia ixx="0.004" ixy="0" ixz="0" iyy="0.004" iyz="0" izz="0.0001"/>
+    </inertial>
+  </link>
+  <joint name="velodyne_mast_joint" type="fixed">
+    <parent link="top_plate_link"/>
+    <child link="velodyne_mast_link"/>
+    <!-- x=-0.50 on the plate (base_link x~-0.42): behind the stow forearm fold
+         (which reaches back to base_link x~-0.23) yet still over the chassis
+         (rear edge ~-0.49). -->
+    <origin xyz="-0.50 0.0 0.0" rpy="0 0 0"/>
+  </joint>
+  <xacro:include filename="$(find velodyne_description)/urdf/VLP-16.urdf.xacro"/>
+  <xacro:VLP-16 parent="velodyne_mast_link" name="velodyne" topic="/velodyne_points"
+                hz="10" samples="1875" gpu="true"
+                min_range="0.5" max_range="100.0">
+    <origin xyz="0.0 0.0 0.40" rpy="0.0 0.0 0.0"/>
+  </xacro:VLP-16>
+  <!-- ===== Dedicated IMU for LiDAR-inertial odometry (gravity-included) =====
+       DLIO/FAST-LIO require the accelerometer to report the gravity reaction
+       (~9.8 m/s² at rest) to estimate orientation + the gravity vector. The
+       stock Husky IMU (libhector_gazebo_ros_imu, topic /imu/data) outputs
+       kinematic acceleration WITHOUT gravity, so LIO init fails. The Gazebo
+       sensor-based libgazebo_ros_imu_sensor reads the true simulated IMU
+       (gravity included). Mounted axis-aligned at the base_link origin so the
+       base_link->imu extrinsic is identity. Topic: /lidar/imu. -->
+  <link name="imu_lidar_link">
+    <inertial>
+      <mass value="0.01"/>
+      <origin xyz="0 0 0" rpy="0 0 0"/>
+      <inertia ixx="1e-6" ixy="0" ixz="0" iyy="1e-6" iyz="0" izz="1e-6"/>
+    </inertial>
+  </link>
+  <joint name="imu_lidar_joint" type="fixed">
+    <parent link="base_link"/>
+    <child link="imu_lidar_link"/>
+    <origin xyz="0 0 0" rpy="0 0 0"/>
+  </joint>
+  <gazebo reference="imu_lidar_link">
+    <sensor name="imu_lidar_sensor" type="imu">
+      <always_on>true</always_on>
+      <update_rate>200</update_rate>
+      <visualize>false</visualize>
+      <plugin name="imu_lidar_plugin" filename="libgazebo_ros_imu_sensor.so">
+        <topicName>/lidar/imu</topicName>
+        <bodyName>imu_lidar_link</bodyName>
+        <frameName>imu_lidar_link</frameName>
+        <updateRateHZ>200.0</updateRateHZ>
+        <gaussianNoise>0.0</gaussianNoise>
+        <initialOrientationAsReference>false</initialOrientationAsReference>
+      </plugin>
+    </sensor>
+  </gazebo>
   <xacro:include filename="$(find ur_description)/urdf/inc/ur_macro.xacro"/>
   <xacro:ur_robot
