Commit message: feat(air-ground): UGV terrain nav on UAV map + UAV global/EGO planner + stability/speed
空地协同：无人机建图 -> 地面车在无人机地图上做地形感知导航与上坡。

UAV 侧（低空建图，绕楼 + 穿树林）
- global_path_planner.py(新增)：A* 全局前端绕大楼；按连通域面积把树滤掉、交给 EGO
  局部避障穿过；纯追踪 + 串拉抽稀让轨迹更直；子目标爬到巡航高度并设最低高度兜底，
  防退化/防原地卡死；反应式贴楼退后默认关（局部避障交给 EGO，避免前后振荡）。
- forest_uav_mapping.launch/forest_param.xml/forest_utils.launch：低空建图参数 + 全局规划接线。
- px4_bridge.py：关闭反应式 depth 拦截，规划权交给 EGO。
- 新增 clean_pcd.py / uav_map_origin_saver.py / coordinate_align_checker.py。

UGV 侧（地形可通行图 + 导航）
- pcd_to_occupancy_map.py(新增)：UAV PCD -> 静态全局占据图；坡度不判障碍、全地面可走
  （仅楼/墙致命），坡度连续着色可视化；GPS/UTM 锚定对齐(sidecar 零配置)。
- terrain_layer.yaml(trinary=false 保留坡度信息)、costmap_common(修激光命名空间让实时
  LiDAR 生效 + 加大膨胀离障碍远)、dwa(提速 + 解决大转弯卡死)、ugv_terrain_nav.launch、
  terrain_nav.rviz。
- 稳定/抓地：urdf 低压舱降重心 + 轮摩擦 mu=3 + UR5 折叠贴车顶行车姿态；平地提速 1.5 m/s。
- ekf_global 3D + Gazebo 真值 z 让车随坡显示；局部 EKF 3D 修坡上激光投影
  （消除 'None of the plan points ... free' 代价图报错）。

文档：PROJECT_PROGRESS.md、docs/(坐标对齐 UTM、运行手册)。
清理：移除指向他人机器 /home/jun 的失效符号链接 etc、test_data。

Co-Authored-By: Claude Opus 4.8 <noreply@anthropic.com>

File: src/mobile_manipulator/urdf/husky_ur5.urdf.xacro (robot description, xacro)
@@ -28,13 +28,16 @@
        The stock inertial_link iyy (1.74 kg⋅m²) is less than half the
        theoretical value for the chassis dimensions, leaving the base on the
-       edge of tipping when the arm is extended.  30 kg placed 0.15 m behind
-       and 0.08 m below base_link shifts the CoM rearward and raises iyy
-       enough to keep the robot stable through the full grasp motion. -->
+       edge of tipping when the arm is extended.  The mass is placed behind and
+       BELOW base_link to shift the CoM rearward and DOWN.
+       上坡稳定性加强：UR5 装在顶板上抬高了整车质心，在斜坡上(尤其转弯/进坡)容易
+       翻车。把压舱质量从 30→45 kg、并从 -0.08 下沉到 -0.20 m(到接触面附近)，显著
+       压低质心 -> 抗倾覆角变大、坡上不易翻。配合 slope_max 限到 ~22° 不去爬超过
+       翻车角的坡，以及 DWA 减速/缓转。 -->
   <link name="base_ballast">
     <inertial>
-      <mass value="30.0" />
-      <origin xyz="-0.15 0.0 -0.08" rpy="0 0 0" />
-      <inertia ixx="1.5" ixy="0" ixz="0"
-               iyy="3.0" iyz="0" izz="3.0" />
+      <mass value="45.0" />
+      <origin xyz="-0.15 0.0 -0.20" rpy="0 0 0" />
+      <inertia ixx="2.5" ixy="0" ixz="0"
+               iyy="4.0" iyz="0" izz="4.0" />
     </inertial>
   </link>
@@ -150,3 +153,40 @@
     </sensor>
   </gazebo>
+  <!-- ===== 地面真值位姿(含真实高度 z)：让 UGV 在 RViz 里跟着地形爬高 =====
+       2D 模式的 EKF 把机器人 z 锁成 0，在真实高程的坡上 UGV 就被埋到坡面下。
+       这个 p3d 插件直接从 Gazebo 取 base_link 的真值位姿(含 z/俯仰)，发到
+       /ground_truth/state，由 global EKF 只融合其中的 z(见 ekf_global.yaml)。
+       frameName=map：本工程 map 原点 == Gazebo 世界原点(GPS 锚定)，故真值世界 z
+       即 map 系 z。只喂 z、不动 x/y(仍由轮速+GPS主导)，对 2D 导航几乎无影响。 -->
+  <gazebo>
+    <plugin name="ground_truth_p3d" filename="libgazebo_ros_p3d.so">
+      <bodyName>base_link</bodyName>
+      <topicName>/ground_truth/state</topicName>
+      <frameName>map</frameName>
+      <updateRate>50.0</updateRate>
+      <gaussianNoise>0.0</gaussianNoise>
+      <xyzOffset>0 0 0</xyzOffset>
+      <rpyOffset>0 0 0</rpyOffset>
+    </plugin>
+  </gazebo>
+  <!-- ===== 上坡力度：加大 4 个驱动轮的接触摩擦 =====
+       stock husky_description/wheel.urdf.xacro 设 mu1=mu2=1.0，仿真里在坡面上
+       轮子打滑 -> 上不去/往下滑（轮关节是 continuous 且无 effort 限制，所以瓶颈
+       是【摩擦】不是扭矩）。这里按轮 link 名再写一遍 <gazebo reference> 覆盖，
+       SDF 取后出现的值 -> mu 提到 3.0，沿滚动方向(fdir1=x)抓地更牢，上坡少打滑。
+       kp/kd 沿用 husky 默认接触刚度。配合压低质心(压舱)+收臂行车姿态一起防打滑/翻车。 -->
+  <xacro:macro name="wheel_friction" params="link">
+    <gazebo reference="${link}">
+      <mu1 value="3.0"/>
+      <mu2 value="3.0"/>
+      <kp value="10000000.0"/>
+      <kd value="1.0"/>
+      <fdir1 value="1 0 0"/>
+      <minDepth>0.005</minDepth>
+    </gazebo>
+  </xacro:macro>
+  <xacro:wheel_friction link="front_left_wheel_link"/>
+  <xacro:wheel_friction link="front_right_wheel_link"/>
+  <xacro:wheel_friction link="rear_left_wheel_link"/>
+  <xacro:wheel_friction link="rear_right_wheel_link"/>
 </robot>

Commit message: fix(grasp): stop the pick throwing the robot, and make the grasp physically possible
The pick threw the 46 kg Husky metres across the world. It turned out to be two
independent causes stacked on top of each other, and both are now measured rather
than guessed.

1. THE CLOSE WAS RAMMING THE BLOCK.
   The SRDF carried a pad-gap curve that was invented: it claimed 40 mm of gap at
   finger_joint=0.537. The truth, by FK from our own URDF (and confirmed to three
   decimals against a teammate's independently measured table), is 40 mm at q~0.495.

       q      0.000   0.400   0.480   0.495   0.500   0.580
       gap   128.5    58.9    43.46   40.53   39.55   23.76  mm

   Read the last column. "closed" was 0.58 -- a 23.76 mm gap around a 40 mm block,
   i.e. 16.2 mm of interpenetration. The 2F-140's mimic joints are driven by
   SetPosition() (a kinematic teleport) and right_outer_knuckle_joint is itself a
   mimic, so the entire right finger is kinematic: it is forced to its commanded
   angle whatever it is touching and exerts NO force. It cannot stall on the block.
   It PENETRATES it, and the solver's answer to that penetration is what ejected the
   mine and threw the robot. That was "the roll".

   So the jaws now close to 0.400 -- a 58.9 mm gap, ~8.6 mm of air per side -- and
   never touch the mine at all. We give up nothing: this gripper has no grip to give.

2. THE ARM WAS LEVERING AN UNBRAKED ROBOT.
   Nobody had measured this. MERELY MOVING THE ARM TO THE GRASP POSE displaced
   base_link by 0.030 m and lifted it 26 mm, with nothing grasped and nothing touched.
   husky_velocity_controller commands wheel VELOCITY and has no position hold, so
   nothing whatsoever resists a 20 kg UR5 cantilevered forward and down at the edge of
   its reachable band. The pick was spending its whole stability budget before it began.

   gazebo_link_attacher (new) welds base_link to the static ground for the duration of
   the pick, released on every exit path. It is also what carries the mine: a friction
   grasp is not available at any commanded angle, so the grasp is an explicit joint,
   verified rigid to 0.1 mm (TCP +0.1500 m, mine +0.1499 m, base +0.0002 m).

gazebo_grasp_fix is REMOVED, and that reverses an earlier decision. It welds only on
two OPPOSING CONTACT FORCES, which a kinematic finger never produces, so it fires on
solver noise instead: across seven trials its "attach" landed at finger_joint 0.4254,
0.4387, 0.4413, 0.480, 0.495 and once at 0.0017 (jaws WIDE OPEN), all for the same
40 mm block. Tightening grip_count_threshold to reject the noise stopped it firing at
the real contact too. Its hold is broken independently: it welds with a model-less
zero-limit revolute, which on Gazebo 11 is a free hinge -- during a lift the TCP rose
120 mm while the mine rose 16 mm.

Also here, from the same effort:
  * mimic_joint_plugin: read PID gains from SDF, not the ROS parameter server. The
    mere PRESENCE of any /gazebo_ros_control/pid_gains/* param makes gzserver abort at
    startup with std::bad_array_new_length. Verified by bisection.
  * robotiq pads: kp 1e5 / kd 100 / mu 1.6. They had Gazebo's default kp ~1e13 -- rigid
    steel. The real pads are rubber.
  * finger_joint path tolerance disabled: a gripper that is holding something
    necessarily falls behind its commanded path, and policing that was aborting the
    pick mid-grasp (PATH_TOLERANCE_VIOLATED: finger_joint path error 0.512).

Measured: base displacement through the entire pick is 0.0000 m, against a 0.03 m gate.

Co-Authored-By: Claude Opus 4.8 <noreply@anthropic.com>

File: src/mobile_manipulator/urdf/husky_ur5.urdf.xacro (robot description, xacro)
@@ -135,28 +135,53 @@
     <origin xyz="0 0 0" rpy="0 -1.57 1.57"/>
   </xacro:robotiq_140_gripper>
-  <!-- Grasp fix: creates a virtual joint between gripper and object when both
-       fingers make opposing contact, preventing the object from flying away. -->
-  <gazebo>
-    <plugin filename="libgazebo_grasp_fix.so" name="gazebo_grasp_fix">
-      <!-- palm_link must be a link that survives Gazebo's fixed-joint lumping.
-           robotiq_arg2f_base_link is attached by a fixed joint and gets merged
-           into the UR5 wrist, so we use ur5_wrist_3_link as the palm (as the
-           Hand-E setup did). The inner_finger links are joined by revolute joints
-           and survive; they also absorb the fixed-jointed finger-pad collisions. -->
-      <arm>
-        <arm_name>robotiq_140</arm_name>
-        <palm_link>ur5_wrist_3_link</palm_link>
-        <gripper_link>left_inner_finger</gripper_link>
-        <gripper_link>right_inner_finger</gripper_link>
-      </arm>
-      <forces_angle_tolerance>100</forces_angle_tolerance>
-      <update_rate>90</update_rate>
-      <grip_count_threshold>1</grip_count_threshold>
-      <max_grip_count>8</max_grip_count>
-      <release_tolerance>0.005</release_tolerance>
-      <disable_collisions_on_attach>false</disable_collisions_on_attach>
-      <contact_topic>__default_topic__</contact_topic>
-    </plugin>
-  </gazebo>
+  <!-- ===== grasp_tcp: THE grasp frame. Every grasp pose is a pose of this link. =====
+       Parented to the gripper (not ur5_tool0) so it is a property of the hand and
+       survives a remount. Its numbers are FK, not guesses: the jaw center-line is by
+       definition the midpoint of the two inner_finger_pads, and that midpoint lies
+       exactly on robotiq_arg2f_base_link's +Z at x=y=0 —
+           finger_joint = 0.000 (open)   -> midpoint z = 0.1770, gap 136.0 mm
+           finger_joint = 0.350          -> midpoint z = 0.1945, gap  75.9 mm
+           finger_joint = 0.695 (closed) -> midpoint z = 0.2007, gap   8.3 mm
+       z = 0.177 = the OPEN jaw center, i.e. where the object sits at the instant the
+       gripper ARRIVES at the grasp (we always approach open). Note the pads then
+       ADVANCE ~21 mm further along +Z as they close — that is the 2F-140's four-bar
+       linkage arc, not an error — so a grasp aimed exactly at an object's center will
+       have the pads settle ~21 mm beyond it. Grasp code compensates by aiming high;
+       for the 60 mm landmine detonator that is comfortably inside the block.
+       AXES (the one convention, defined once, used everywhere):
+           +Z = approach        (out of the palm, between the fingers)
+           +X = finger closing  (== GPD's `binormal`)
+           +Y = GPD's `axis`
+       The gripper base's own axes are +Z approach / +-Y closing, so this is a pure
+       +90 deg yaw: Rz(pi/2) sends tcp_X -> base_Y (closing) and leaves tcp_Z = base_Z.
+       This link replaces the legacy scalars GPD_TOOL_OFFSET=0.12 and FINGER_REACH=0.18,
+       which tried to fake a grasp frame by sliding ur5_tool0 along tool0's OWN +Z — but
+       the gripper is mounted rpy="0 -1.57 1.57", so tool0's Z is not the approach axis
+       at all. Set MoveIt/MTC ik_frame to grasp_tcp and the offsets vanish.
+       Massless and geometry-less: Gazebo lumps it away, so it adds no physics and needs
+       no SRDF collision entry. -->
+  <link name="grasp_tcp"/>
+  <joint name="grasp_tcp_joint" type="fixed">
+    <parent link="robotiq_arg2f_base_link"/>
+    <child  link="grasp_tcp"/>
+    <origin xyz="0 0 0.177" rpy="0 0 ${pi/2}"/>
+  </joint>
+  <!-- gazebo_grasp_fix IS DELIBERATELY NOT LOADED. It cannot work on this gripper, and
+       leaving it running would fight the weld that does.
+       It attaches an object only when it sees TWO OPPOSING CONTACT FORCES on the finger links.
+       But the 2F-140's mimic joints are all driven by robotiq_gazebo's MimicJointPlugin via
+       SetPosition(), a kinematic teleport, and right_outer_knuckle_joint is itself a mimic,
+       so the ENTIRE right finger is kinematic: forced to its commanded angle regardless of what
+       it touches, exerting no force on anything. There are no opposing grip forces here for
+       grasp_fix to find, so it fires on solver noise instead. Measured across 7 trials, its
+       "attach" landed at finger_joint = 0.4254, 0.4387, 0.4413, 0.480, 0.495 and even 0.0017
+       (jaws WIDE OPEN) for one and the same 40 mm block, whose true contact angle is 0.495.
+       Raising grip_count_threshold to reject that noise stopped it firing at the real contact
+       too. Its hold is broken independently: it welds with a MODEL-LESS ZERO-LIMIT REVOLUTE,
+       which on Gazebo 11 is a free hinge. During a lift the TCP rose 120 mm while the mine
+       rose 16 mm, and the constraint reaction jacked the 46 kg base into the air.
+       The grasp is therefore an EXPLICIT WELD (gazebo_link_attacher, registered in
+       outdoor_city.world): the jaws close to a gap slightly WIDER than the block so they never
+       touch it, and a real fixed joint carries it. See grasp_mtc/scripts/grasp_task.py. -->
   <link name="realsense_camera_link">
     <visual>

File: src/robotiq/robotiq_description/urdf/robotiq_140_gripper.urdf.xacro (robot description, xacro)
@@ -158,4 +158,20 @@
     <gazebo reference="${prefix}${fingerprefix}_inner_finger_pad">
       <material>Gazebo/Black</material>
+      <!-- These pads are the ONLY surfaces that touch the object, and without these params
+           they inherit Gazebo's default kp of about 1e13: a rigid steel pad. Closing a rigid
+           pad onto a rigid detonator makes the contact ring, which shakes the whole arm and
+           can tip the Husky. The real 2F-140 pads are rubber, so model them as such.
+             kp 1e5 / kd 100 : compliant and heavily damped, absorbing the closing impulse
+             mu 1.6          : rubber on plastic. The grip comes from FRICTION, not from
+                               crushing the object (see the effort limit below)
+             maxVel 0        : never resolve penetration by launching the object
+             minDepth 0.001  : tolerate 1 mm of penetration before reacting, so micro jitter
+                               does not generate impulses -->
+      <mu1>1.6</mu1>
+      <mu2>1.6</mu2>
+      <kp>1e5</kp>
+      <kd>100.0</kd>
+      <maxVel>0.0</maxVel>
+      <minDepth>0.001</minDepth>
     </gazebo>
   </xacro:macro>
@@ -203,5 +219,19 @@
       <child link="${prefix}left_outer_knuckle" />
       <axis xyz="-1 0 0" />
-      <limit lower="0" upper="0.725" velocity="2.0" effort="1000" />
+      <!-- THE GRIP FORCE. gazebo_ros_control drives this position joint with SetPosition()
+           bounded by joint->SetParam("fmax", 0, <this effort limit>), so this number IS the
+           pinch force, and it must be SMALL.
+           Do the arithmetic before changing it. The 2F-140's four-bar gives the pad roughly a
+           0.06 m moment arm, so fingertip force ~ effort / 0.06:
+               effort=1000 (stock) -> ~17000 N. Bulldozes the object; no contact ever forms.
+               effort=20           -> ~330 N.   Still a crowbar: closing on the rigid 40 mm
+                                                detonator injects an impulse that makes the
+                                                jaws buzz and can FLIP THE 46 kg HUSKY.
+               effort=3            -> ~50 N.    What we use.
+           Holding a 0.30 kg mine needs mu*N*2 >= m*g = 2.9 N, i.e. N >= ~1.5 N at mu=1.0.
+           50 N is a 30x margin. There is nothing to buy by going higher, and stability to
+           lose: grip force here is a CONTACT IMPULSE, and the arm is bolted to a wheeled
+           base that can be pushed over by it. -->
+      <limit lower="0" upper="0.725" velocity="2.0" effort="8" />
     </joint>
     <xacro:finger_joints prefix="${prefix}" fingerprefix="left" reflect="1.0"/>
@@ -236,5 +266,25 @@
     <xacro:right_outer_knuckle_joint prefix="${prefix}"/>
     <xacro:robotiq_arg2f_transmission prefix="${prefix}"/>
-    <!-- Mimic joints -->
+    <!-- ===== Mimic joints =====
+         The plugin drives each mimic with SetPosition(), which is a KINEMATIC override, and
+         then bounds it with joint->SetParam("fmax", 0, maxEffort). fmax is what decides
+         whether the linkage can stall on a grasped object or simply drives through it, and
+         the plugin's stock default is maxEffort = 1.0 N.m, which is nowhere near enough to
+         hold the four-bar against contact. We raise it to 20 N.m to match finger_joint's
+         (also newly bounded) effort limit, so the whole linkage stalls together.
+         This matters because the inner_finger joints carry the finger PADS: whatever governs
+         them governs whether the pads can push on an object at all, and therefore whether
+         gazebo_grasp_fix (which attaches only on OPPOSING CONTACT FORCES) can ever fire.
+         The plugin also has a <hasPID/> mode that would drive the mimics with SetForce, which
+         is the more principled option. It is NOT used, for two reasons:
+           1. It was DEAD CODE in this fork: UpdateChild() computed the effort and then threw
+              it away, never calling SetForce. (Fixed anyway in
+              robotiq_gazebo/src/mimic_joint_plugin.cpp, which now applies it and reads its
+              gains from SDF <p>/<i>/<d>.)
+           2. It instantiates a control_toolbox PID inside gzserver, and on this Noetic build
+              ANY control_toolbox PID inside gzserver aborts it at startup with
+              std::bad_array_new_length. Bisected repeatedly. Same for
+              /gazebo_ros_control/pid_gains/* and for effort_controllers.
+         So hasPID stays off until that environment bug is understood. -->
     <gazebo>
       <plugin filename="libgazebo_mimic_joint_plugin.so" name="${prefix}mimic_robotiq_140_1">
@@ -243,4 +293,5 @@
         <multiplier>-1.0</multiplier>
         <offset>0.0</offset>
+        <maxEffort>8.0</maxEffort>
       </plugin>
       <plugin filename="libgazebo_mimic_joint_plugin.so" name="${prefix}mimic_robotiq_140_2">
@@ -249,4 +300,5 @@
         <multiplier>-1.0</multiplier>
         <offset>0.0</offset>
+        <maxEffort>8.0</maxEffort>
       </plugin>
       <plugin filename="libgazebo_mimic_joint_plugin.so" name="${prefix}mimic_robotiq_140_3">
@@ -255,4 +307,5 @@
         <multiplier>-1.0</multiplier>
         <offset>0.0</offset>
+        <maxEffort>8.0</maxEffort>
       </plugin>
       <plugin filename="libgazebo_mimic_joint_plugin.so" name="${prefix}mimic_robotiq_140_4">
@@ -261,4 +314,5 @@
         <multiplier>1.0</multiplier>
         <offset>0.0</offset>
+        <maxEffort>8.0</maxEffort>
       </plugin>
       <plugin filename="libgazebo_mimic_joint_plugin.so" name="${prefix}mimic_robotiq_140_5">
@@ -267,4 +321,5 @@
         <multiplier>1.0</multiplier>
         <offset>0.0</offset>
+        <maxEffort>8.0</maxEffort>
       </plugin>
     </gazebo>

File: src/robotiq/robotiq_description/urdf/robotiq_arg2f_transmission.xacro (robot description, xacro)
@@ -1,4 +1,24 @@
 <?xml version="1.0"?>
 <robot xmlns:xacro="http://ros.org/wiki/xacro">
+  <!-- PositionJointInterface, deliberately. THE GRIP COMES FROM fmax, NOT FROM THE INTERFACE.
+       Read this before "fixing" it to EffortJointInterface.
+       gazebo_ros_control drives a position-mode joint with SetPosition(), but it first calls
+           joint->SetParam("fmax", 0, <URDF effort limit>)
+       and that fmax bounds the force the joint may use to reach its target. With the stock
+       effort="1000" the joint has effectively unlimited authority and simply bulldozes the
+       fingers through whatever is between them. Measured on the 40 mm landmine detonator:
+       finger_joint reached its commanded 0.556 exactly (a 40 mm block should have stalled it
+       near 0.44), Gazebo's contact manager saw NOTHING, gazebo_grasp_fix (which attaches only
+       on OPPOSING CONTACT FORCES) never fired once, and the mine never moved at all.
+       So the fix is to BOUND the effort, not to change the interface: finger_joint's limit is
+       now effort="20" (see robotiq_140_gripper.urdf.xacro), letting the joint stall on the
+       object so real contact forces develop.
+       Why not EffortJointInterface, the textbook answer? Because it forces a control_toolbox
+       PID into the loop (effort_controllers/JointTrajectoryController requires `gains:`), and
+       on THIS Noetic build any control_toolbox PID instantiated inside gzserver aborts it with
+       std::bad_array_new_length. Bisected repeatedly: PID present => gzserver dies at startup
+       every time; PID absent => starts every time. The same applies to
+       /gazebo_ros_control/pid_gains/* and to the mimic plugin's <hasPID/> mode. Until that is
+       diagnosed, PID-based force control is not available in this environment. -->
   <xacro:macro name="robotiq_arg2f_transmission" params="prefix">
     <transmission name="${prefix}finger_joint_trans">
