Commit message: feat: share UAV-to-UGV mine removal pipeline

File: src/mobile_manipulator/urdf/husky_ur5.urdf.xacro (robot description, xacro)
@@ -1,4 +1,12 @@
 <?xml version="1.0"?>
 <robot name="husky_ur5" xmlns:xacro="http://ros.org/wiki/xacro">
+  <!-- Project-owned wrist RGB-D horizontal field of view, in radians.
+       Default 1.308996939 rad = 75 deg.  The previous 60 deg view put the
+       measured M004 detonator ray near v=453/480, behind the gripper crossbar.
+       Widening the optics moves that same ~21 deg ray to v~400 while preserving
+       the camera pose, 640x480 registration, depth geometry and optical frame.
+       This parameter affects visibility only; it is never a grasp target or a
+       substitute for wrist RGB-D measurement. -->
+  <xacro:arg name="wrist_camera_horizontal_fov_rad" default="1.308996939"/>
   <xacro:include filename="$(find husky_description)/urdf/husky.urdf.xacro" />
   <xacro:include filename="$(find husky_description)/urdf/accessories/sick_lms1xx_mount.urdf.xacro" />
@@ -56,4 +64,17 @@
     <origin xyz="0 0 0" rpy="0 -1.57 1.57"/>
   </xacro:robotiq_140_gripper>
+  <!-- Mine-grasp TCP derived from the Robotiq 2F-140 URDF geometry, not from
+       a task-space offset.  At the nominal finger_joint=0.499 rad contact
+       configuration (39.742 mm inner gap for the 40 mm detonator),
+       the two pad centres measured in robotiq_arg2f_base_link are
+       y=+/-0.023621 m, z=0.198591 m.  Their midpoint is therefore the physical
+       contact centre below.  Rz(+pi/2) maps TCP +X onto the jaw-closing axis
+       (gripper-base +Y), while TCP +Z remains the physical approach axis. -->
+  <link name="grasp_tcp"/>
+  <joint name="grasp_tcp_joint" type="fixed">
+    <parent link="robotiq_arg2f_base_link"/>
+    <child link="grasp_tcp"/>
+    <origin xyz="0 0 0.1985905960" rpy="0 0 1.5707963268"/>
+  </joint>
   <!-- Grasp fix: creates a virtual joint between gripper and object when both
        fingers make opposing contact, preventing the object from flying away. -->
@@ -74,8 +95,31 @@
       <update_rate>90</update_rate>
       <grip_count_threshold>1</grip_count_threshold>
-      <max_grip_count>8</max_grip_count>
-      <release_tolerance>0.005</release_tolerance>
-      <disable_collisions_on_attach>false</disable_collisions_on_attach>
+      <!-- Keep the physical opposing-contact requirement, but give an already
+           established grasp 0.5 s of solver-contact hysteresis.  Eight ticks
+           (89 ms) detached one measured grasp during the 3 s hold even though
+           the jaw/TCP relative pose remained inside the executor gate.  The
+           10 mm release displacement is still far below the >50 mm pad motion
+           produced by the verified OPEN command, so PLACE releases normally. -->
+      <max_grip_count>45</max_grip_count>
+      <release_tolerance>0.010</release_tolerance>
+      <!-- Once grasp-fix owns the rigid transport joint, continuing to solve
+           finger/object contacts over-constrains Gazebo and made the measured
+           finger velocity oscillate at 0.27 rad/s.  Disable only the attached
+           object's Gazebo contacts while that joint exists; HandleDetach
+           restores collide mode "all" at PLACE.  MoveIt's attached collision
+           object remains active for arm/chassis planning throughout. -->
+      <disable_collisions_on_attach>true</disable_collisions_on_attach>
       <contact_topic>__default_topic__</contact_topic>
+      <!-- Mission-only simulator fallback. The executor may request this only
+           after its final visual TCP gate and unique spatial association pass.
+           The plugin keeps the same Gazebo model visible as a kinematic palm
+           follower, so it cannot drop or transmit terrain impulses to the UGV. -->
+      <force_lock_enabled>true</force_lock_enabled>
+      <force_attach_topic>/mine_grasp/force_attach</force_attach_topic>
+      <force_detach_topic>/mine_grasp/force_detach</force_detach_topic>
+      <force_status_topic>/mine_grasp/force_lock_status</force_status_topic>
+      <force_arm_name>robotiq_140</force_arm_name>
+      <force_object_prefix>landmine</force_object_prefix>
+      <force_collision_suffix>body::detonator_collision</force_collision_suffix>
     </plugin>
   </gazebo>
@@ -126,5 +170,5 @@
       <visualize>true</visualize>
       <camera>
-        <horizontal_fov>1.047198</horizontal_fov>
+        <horizontal_fov>$(arg wrist_camera_horizontal_fov_rad)</horizontal_fov>
         <image>
           <width>640</width>

File: src/robotiq/robotiq_description/urdf/robotiq_140_gripper.urdf.xacro (robot description, xacro)
@@ -175,4 +175,5 @@
       <axis xyz="1 0 0" />
       <limit lower="-0.8757" upper="0.8757" velocity="2.0" effort="1000" />
+      <dynamics damping="0.05" friction="0.01" />
       <mimic joint="${prefix}finger_joint" multiplier="-1" offset="0" />
     </joint>
@@ -185,4 +186,5 @@
       <axis xyz="1 0 0" />
       <limit lower="-0.8757" upper="0.8757" velocity="2.0" effort="1000" />
+      <dynamics damping="0.05" friction="0.01" />
       <mimic joint="${prefix}finger_joint" multiplier="1" offset="0" />
     </joint>
@@ -204,4 +206,5 @@
       <axis xyz="-1 0 0" />
       <limit lower="0" upper="0.725" velocity="2.0" effort="1000" />
+      <dynamics damping="0.05" friction="0.01" />
     </joint>
     <xacro:finger_joints prefix="${prefix}" fingerprefix="left" reflect="1.0"/>
@@ -214,5 +217,6 @@
       <axis xyz="1 0 0" />
       <limit lower="-0.725" upper="0.725" velocity="2.0" effort="1000" />
-    <mimic joint="${prefix}finger_joint" multiplier="-1" offset="0" />
+      <dynamics damping="0.05" friction="0.01" />
+      <mimic joint="${prefix}finger_joint" multiplier="-1" offset="0" />
     </joint>
     <xacro:finger_joints prefix="${prefix}" fingerprefix="right" reflect="-1.0"/>
@@ -236,5 +240,9 @@
     <xacro:right_outer_knuckle_joint prefix="${prefix}"/>
     <xacro:robotiq_arg2f_transmission prefix="${prefix}"/>
-    <!-- Mimic joints -->
+    <!-- Mimic joints.  A 0.5 mrad deadband suppresses Gazebo constraint noise
+         at a stationary hold without changing the commanded jaw geometry (the
+         corresponding pad displacement is well below one millimetre).  The
+         former 0.1 mrad threshold repeatedly reset all five follower joints and
+         was visible as continuous finger chatter while the arm was moving. -->
     <gazebo>
       <plugin filename="libgazebo_mimic_joint_plugin.so" name="${prefix}mimic_robotiq_140_1">
@@ -243,4 +251,5 @@
         <multiplier>-1.0</multiplier>
         <offset>0.0</offset>
+        <sensitiveness>0.0005</sensitiveness>
       </plugin>
       <plugin filename="libgazebo_mimic_joint_plugin.so" name="${prefix}mimic_robotiq_140_2">
@@ -249,4 +258,5 @@
         <multiplier>-1.0</multiplier>
         <offset>0.0</offset>
+        <sensitiveness>0.0005</sensitiveness>
       </plugin>
       <plugin filename="libgazebo_mimic_joint_plugin.so" name="${prefix}mimic_robotiq_140_3">
@@ -255,4 +265,5 @@
         <multiplier>-1.0</multiplier>
         <offset>0.0</offset>
+        <sensitiveness>0.0005</sensitiveness>
       </plugin>
       <plugin filename="libgazebo_mimic_joint_plugin.so" name="${prefix}mimic_robotiq_140_4">
@@ -261,4 +272,5 @@
         <multiplier>1.0</multiplier>
         <offset>0.0</offset>
+        <sensitiveness>0.0005</sensitiveness>
       </plugin>
       <plugin filename="libgazebo_mimic_joint_plugin.so" name="${prefix}mimic_robotiq_140_5">
@@ -267,4 +279,5 @@
         <multiplier>1.0</multiplier>
         <offset>0.0</offset>
+        <sensitiveness>0.0005</sensitiveness>
       </plugin>
     </gazebo>
